File: sigmabot.kicad_pcb (KiCad board)
At the start: 2 copper layers, 223 x 111 mm, 14 parts, among them J1 Conn_01x02, J2 Conn_01x07, J3 MOTOR_L, J4 MOTOR_R, SW1 SW_DPDT_x2, U1 BUCK_CONV

Commit message: Just opened and closed it in newest kicad and it updated the PCB.
Other:
- net class Default removed
